File: eagle/EspressoWemos/EspressoWemos.brd (EAGLE design)
At the start: 33.3 x 25.5 mm, 28 parts, among them Q1 MMBT2222A, Q2 MMBT2222A, U1 mux

Commit message: Updated eagle files
Parts:
- added J1: RJ45, SparkFun-Connectors:RJ45-8
- R7, R8: value 3.3K -> 6.6K
Changed lines of the file:
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@@
 <attribute name="PROD_ID" value="TRANS-08049" x="-26.67" y="90.17" size="1.778" layer="28" rot="MR180" display="off"/>
 </element>
-<element name="R7" library="rcl" package="R1206" value="3.3K" x="66.04" y="54.61" rot="MR90"/>
-<element name="R8" library="rcl" package="R1206" value="3.3K" x="55.88" y="69.85" rot="R270"/>
+<element name="R7" library="rcl" package="R1206" value="6.6K" x="66.04" y="54.61" rot="MR90"/>
+<element name="R8" library="rcl" package="R1206" value="6.6K" x="55.88" y="69.85" rot="R270"/>
 <element name="R9" library="rcl" package="R1206" value="10K" x="54.61" y="71.12" rot="MR0"/>
 <element name="R10" library="rcl" package="R1206" value="150" x="45.72" y="59.69" rot="MR0"/>
@@
 <element name="R13" library="rcl" package="R1206" value="150" x="39.37" y="59.69" rot="MR0"/>
 <element name="R14" library="rcl" package="R1206" value="10K" x="66.04" y="58.42" rot="R90"/>
+<element name="J1" library="SparkFun-Connectors" package="RJ45-8" value="RJ45" x="26.67" y="63.5">
+<attribute name="PROD_ID" value="CONN-08506" x="26.67" y="63.5" size="1.778" layer="27" display="off"/>
+</element>
 </elements>
 <signals>
