File: eagle/EspressoWemos/EspressoWemos.sch (EAGLE design)
At the start: 28 parts, among them Q1 MMBT2222A, Q2 MMBT2222A, U1 mux

Commit message: Updated eagle files
Parts:
- added J1: RJ45, SparkFun-Connectors:RJ45-8PTH
- R7, R8: value 3.3K -> 6.6K
Changed lines of the file:
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@@
 <part name="Q1" library="SparkFun-DiscreteSemi" deviceset="TRANSISTOR_NPN" device="MMBT2222A" value="MMBT2222A"/>
 <part name="Q2" library="SparkFun-DiscreteSemi" deviceset="TRANSISTOR_NPN" device="MMBT2222A" value="MMBT2222A"/>
-<part name="R7" library="rcl" deviceset="R-US_" device="R1206" value="3.3K"/>
-<part name="R8" library="rcl" deviceset="R-US_" device="R1206" value="3.3K"/>
+<part name="R7" library="rcl" deviceset="R-US_" device="R1206" value="6.6K"/>
+<part name="R8" library="rcl" deviceset="R-US_" device="R1206" value="6.6K"/>
 <part name="R9" library="rcl" deviceset="R-US_" device="R1206" value="10K"/>
 <part name="R10" library="rcl" deviceset="R-US_" device="R1206" value="150"/>
@@
 <part name="R13" library="rcl" deviceset="R-US_" device="R1206" value="150"/>
 <part name="R14" library="rcl" deviceset="R-US_" device="R1206" value="10K"/>
+<part name="J1" library="SparkFun-Connectors" deviceset="RJ45-8" device="PTH" value="RJ45"/>
 </parts>
 <sheets>
@@
 <instance part="R13" gate="G$1" x="149.86" y="88.9" rot="R180"/>
 <instance part="R14" gate="G$1" x="170.18" y="73.66" rot="R270"/>
+<instance part="J1" gate="JP1" x="276.86" y="124.46"/>
 </instances>
 <busses>
